File: Lora puck.kicad_sch (KiCad schematic)
At the start: 10 parts, among them J1 USB_C_Receptacle_USB2.0_16P, SW1 SW_Push, U1 RP2040, U2 AP2112K-3.3

Commit message: Add files via upload
Parts:
- added C10, C13: 1uF, symbol Device:C
- added C11, C12, C14, C15, C2, C3, C4, C5, C6, C7, C8, C9: 100nF, symbol Device:C
- added C16, C17: 33pf, symbol Device:C
- added C18: 47nF, symbol Device:C
- added C19: 47pF, symbol Device:C
- added C20, C26: Unpopulated, symbol Device:C
- added C21: 5.6pF, symbol Device:C
- added C22, C29, C30: 3.3pF, symbol Device:C
- added C23, C28: 39pF, symbol Device:C
- added C24: 2.2pF, symbol Device:C
- added C25: 2.4pF, symbol Device:C
- added C27: 1.8pF, symbol Device:C
- added C31, C32: 1nF, symbol Device:C
- added IC1: PE4259-63, SOT65P210X110-6N, symbol Rf_Switch:PE4259-63
- added J2: Conn_Coaxial, symbol Connector:Conn_Coaxial
- added L1: 47nH, symbol Device:L
- added L2: 0, symbol Device:L
- added L3: 2.5nH, symbol Device:L
- added L4: 4.7nH, symbol Device:L
- added L5: 15nH, symbol Device:L
- added L6: 9.1nH, symbol Device:L
- added R6: 10k, symbol Device:R
- added R7, R8: 100R, symbol Device:R
- added U3: W25Q128JVS, Package_SO:SOIC-8_5.3x5.3mm_P1.27mm, symbol Memory_Flash:W25Q128JVS
- added U4: SX1262IMLTRT, Package_DFN_QFN:QFN-24-1EP_4x4mm_P0.5mm_EP2.6x2.6mm, symbol RF:SX1262IMLTRT
- added Y1: Crystal_GND24, symbol Device:Crystal_GND24
Connections:
- net +3.3V: now also C10.1, C11.1, C12.1, C14.1, C15.1, C2.1, C3.1, C4.1, C5.1, C6.1, C7.1, R6.1, U3.8 (VCC), U4.1 (VDD_IN), U4.10 (VBAT), U4.11 (VBAT_IO)
- net GND: now also U1.19 (TESTEN), C10.2, C11.2, C12.2, C13.2, C14.2, C15.2, C16.1, C17.2, C18.2, C19.2, C2.2, C20.2, C21.2, C24.2, C26.2, C27.2, C29.2, C3.2, C30.2, C31.2, C32.2, C4.2, C5.2, C6.2, C7.2, C8.2, C9.2, IC1.2 (GND), J2.2 (Ext), U3.4 (GND), U4.2 (GND), U4.20 (GND), U4.25 (GND), U4.5 (GND), U4.8 (GND), Y1.2, Y1.3
- net XIN: now reaches U1.20 (XIN)
- net XIN: now also C16.2, Y1.1
- net XOUT: now reaches U1.21 (XOUT)
- net XOUT: now also C17.1, Y1.4
- net BUSY: now reaches U1.34 (GPIO22)
- net BUSY: now also U4.14 (BUSY)
- net IO3: now reaches U1.51 (QSPI_SD3)
- net IO3: now also U3.7 (~{HOLD}/~{RESET}/IO_{3})
- net CLK: now reaches U1.52 (QSPI_SCLK)
- net CLK: now also U3.6 (CLK)
- net I0O: now reaches U1.53 (QSPI_SD0)
- net IO2: now reaches U1.54 (QSPI_SD2)
- net IO2: now also U3.3 (~{WP}/IO_{2})
- net IO1: now reaches U1.55 (QSPI_SD1)
- net IO1: now also U3.2 (DO/IO_{1})
- net /CS: now reaches U1.56 (QSPI_SS)
- net /CS: now also R6.2, U3.1 (~{CS})
- new net: C25.2, C26.1, IC1.3 (RF2)
- new net: C24.1, IC1.1 (RF1), L4.2
- new net: C32.1, IC1.4 (CTRL), R8.1
- new net: C28.1, IC1.5 (RFC)
- new net: C31.1, IC1.6 (~{CTRL_OR_VDD}), R7.1
- new net: C28.2, C29.1, L6.1
- new net: C20.1, C22.1, L1.2, L2.2, L3.1
- new net: C21.1, C22.2, C23.1, L3.2
- new net: C30.1, J2.1 (In), L6.2
- new net: C23.2, L4.1
- new net +1V1: C13.1, C8.1, C9.1
- new net DIO2: R7.2, R8.2, U4.12 (DIO2)
- new net IO0: U3.5 (DI/IO_{0})
- new net RFI_N: C25.1, L5.2, U4.22 (RFI_N)
- new net RFI_P: C27.1, L5.1, U4.21 (RFI_P)
- new net RFO: L2.1, U4.23 (RFO)
- new net VR_PA: C18.1, C19.1, L1.1, U4.24 (VR_PA)
Other:
- note added: "ADC_AVDD"
- note added: "Crystal X322512MSB4SI"
- note added: "DVDD Decoupling"
- note added: "Flash memory"
- note added: "IOVDD Decoupling"
- note added: "Microcontroller"
- note added: "Quad QSPI Flash"
- note added: "USB_C power"
- note added: "USB_VDD"
- note added: "VREG_VIN"
- note added: "VREG_VOUT"
- moved on the sheet: C1, J1, R1, R2, R3, R4, R5, SW1, U1, U2
